File: hardware/display.kicad_sch (KiCad schematic)
At the start: 7 parts

Commit message: finalize fab files
Parts:
- U?: footprint matei:GC9A01Round1.28 -> matei:GC9A01Round1.28_flipped_mount_easy_esc
Changed lines of the file:
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@@
       (effects (font (size 1.27 1.27)) (justify left))
     )
-    (property "Footprint" "matei:GC9A01Round1.28" (at 154.94 95.25 0)
+    (property "Footprint" "matei:GC9A01Round1.28_flipped_mount_easy_esc" (at 154.94 95.25 0)
       (effects (font (size 1.27 1.27)) hide)
     )
-    (property "Datasheet" "" (at 132.08 90.17 0)
+    (property "Datasheet" "" (at 132.08 90.17 0) (show_name)
       (effects (font (size 1.27 1.27)) hide)
     )

Commit message: update schematic to remove debounce cap
Parts:
- U?: now left out of the parts list
Changed lines of the file:
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@@
   )
   (symbol (lib_id "matei:GC9A01") (at 132.08 90.17 0) (unit 1)
-    (in_bom yes) (on_board yes) (dnp no)
+    (in_bom no) (on_board yes) (dnp no)
     (property "Reference" "U?" (at 123.19 77.47 0)
       (effects (font (size 1.27 1.27)) (justify left))
